File: crates/gcode-kicad/tests/fixtures/circuits/mosfet-switch.kicad_sch (KiCad schematic)
At the start: 5 parts, among them Q1 Q_NMOS_GSD

Commit message: KiCad 10: real ERC 10/10 PASS, v10 format tokens, fix symbol-library drift
Environment moved to KiCad 10.0.7, which unblocked tasks 1.1/1.2 and surfaced a
real defect:

- catalog: Device:Q_NMOS_GSD no longer exists in KiCad 10; the replacement
  Device:Q_NMOS uses LETTER pin numbers (D/G/S). The stale entry silently fell
  back to the 2-pin generic stub, and the stub made ERC report PASS - a false
  pass. Fixed, plus two guard tests (every lib_id must resolve; every referenced
  pin must exist on its symbol) and the acceptance harness now refuses to count
  a stub-substituted circuit (exit 4).
- schematic: emit the KiCad 10 format (version 20260306, generator_version 10.0,
  quoted uuids, body_style/exclude_from_sim/in_pos_files, (hide yes) property
  form) so the declared format matches the embedded v10 symbol definitions.
- fixtures regenerated; 89 tests green
- KR1: 10/10 on all four measurable tracks (generate, symbol resolution,
  KiCad netlist exact, ERC PASS) vs target >= 7
- docs: PRD appendix and tasks.md updated; 44/44 tasks complete
Parts:
- removed Q1: Q_NMOS_GSD, symbol Device:Q_NMOS_GSD
- added Q1: Q_NMOS, symbol Device:Q_NMOS
Connections:
- net DRAIN: now also Q1.D
- net GATE: now also Q1.G
- net GND: now also Q1.S
